File: 2Inputs.kicad_sch (KiCad schematic)
At the start: 14 parts, among them J1 JST_SH_SM06B-SRSS-TB_1x06-1MP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, J2 Input0, J3 Input1, J4 Conn_01x04, U1 M24C02-FMN

Commit message: Change screw terminals to 3.5mm version
Parts:
- J2, J3: footprint TerminalBlock_TE-Connectivity:TerminalBlock_TE_282834-2_1x02_P2.54mm_Horizontal -> TerminalBlock_4Ucon:TerminalBlock_4Ucon_1x02_P3.50mm_Horizontal
- J4: footprint Connector_PinSocket_2.54mm:PinSocket_1x04_P2.54mm_Vertical -> Library:PogoPinsPads_1x04_P2.5mm
Changed lines of the file:
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@@
 			)
 		)
-		(property "Footprint" "TerminalBlock_TE-Connectivity:TerminalBlock_TE_282834-2_1x02_P2.54mm_Horizontal"
+		(property "Footprint" "TerminalBlock_4Ucon:TerminalBlock_4Ucon_1x02_P3.50mm_Horizontal"
 			(at 34.29 33.02 0)
 			(effects
@@
 			)
 		)
-		(property "Footprint" "Connector_PinSocket_2.54mm:PinSocket_1x04_P2.54mm_Vertical"
+		(property "Footprint" "Library:PogoPinsPads_1x04_P2.5mm"
 			(at 156.21 71.12 0)
 			(effects
@@
 			)
 		)
-		(property "Footprint" "TerminalBlock_TE-Connectivity:TerminalBlock_TE_282834-2_1x02_P2.54mm_Horizontal"
+		(property "Footprint" "TerminalBlock_4Ucon:TerminalBlock_4Ucon_1x02_P3.50mm_Horizontal"
 			(at 34.29 59.69 0)
 			(effects
